Commit message: New working moveit_configs (cell_test) Changed: /..support/urdf/cell.xacro controller_manager.launch planning_execution.launch planning_context.launch controllers.yaml

File: kappers_pakker_support/urdf/cell.xacro (robot description, xacro)
@@ -32,3 +32,9 @@
         <origin xyz="0 0 0" rpy="0 0 0"/>
     </joint>
+    <!-- Connect tool0_controller to base using floating joint -->
+    <joint name="base-tool0_controller_floating_joint" type="floating">
+      <origin xyz="0 0 0" rpy="0 0 0"/>
+      <parent link="base"/>
+      <child link="tool0"/>
+    </joint>
 </robot>
