Commit message: Ur_manager now has access to throw service - unstable but works!

File: ur_related/ur_manager_support/urdf/ur5_throw_cell.xacro (robot description, xacro)
@@ -1,4 +1,2 @@
-<<<<<<< HEAD:ur_manager_support/urdf/ur5_throw_cell.urdf
-=======
 <?xml version="1.0" ?>
 <robot name="ur5_throw_cell" xmlns:xacro="http://ros.org/wiki/xacro">
@@ -146,4 +144,20 @@
         </collision>
     </link>
+    <link name="dummy_grippers">
+        <visual>
+            <geometry>
+                <box size="0.14 0.03 0.095" />
+            </geometry>
+            <material name="pale_green">
+                <color rgba="0.1 1.0 0 0.8" />
+            </material>
+        </visual>
+        <collision>
+            <origin xyz="0 0 0" rpy="0 0 0" />
+            <geometry>
+                <box size="0.14 0.03 0.095" />
+            </geometry>
+        </collision>
+    </link>
     <joint name="gripper_disc_to_robot" type="fixed">
         <origin xyz="0.01 0 0" rpy="0 ${pi/2} 0"/>
@@ -152,4 +166,5 @@
     </joint>
     <xacro:wsg_50_xacro name="wsg" parent="gripper_disc" finger_length="0.048" finger_tip="0.004">
+   <!-- finger_length="0.048" finger_tip="0.004"  (original model)-->
         <origin xyz="0 0 0.01" rpy="${pi} -${pi} -${pi/2}"/>
     </xacro:wsg_50_xacro>
@@ -159,4 +174,9 @@
         <child link="gripper_plugs"/>
     </joint>
+    <joint name="dummy_grippers_to_wsg" type="fixed">
+        <origin xyz="0 0 0.08" rpy="0 0 0"/>
+        <parent link="wsg_center"/>
+        <child link="dummy_grippers"/>
+    </joint>
     <!-- ***JOINTS*** -->
     <joint name="table_top_to_world" type="fixed">
@@ -186,5 +206,5 @@
     </joint>
     <joint name="camera_to_post_top" type="fixed">
-        <origin xyz="-0.041 -0.024 0" rpy="${pi/2} 0 0"/>
+        <origin xyz="-0.041 -0.024 -0.01" rpy="${pi/2} 0 0"/> <!--IS BEING TWEEKED-->
         <parent link="post_top"/>
         <child link="camera"/>
@@ -230,3 +250,2 @@
 </joint>
 -->
->>>>>>> 26a60b4c68b3a2a261a9b928b81953632d92833b:ur_related/ur_manager_support/urdf/ur5_throw_cell.xacro

Commit message: Picker node V1 finished - will terminate throw routine if one srv fails! - publishes times

File: ur_related/ur_manager_support/urdf/ur5_throw_cell.xacro (robot description, xacro)
@@ -24,5 +24,5 @@
             <origin xyz="0 0 0" rpy="0 0 0" />
             <geometry>
-                <box size="1.4 1.45 0.75" />
+                <box size="1.45 1.4 0.75" />
             </geometry>
         </collision>

Commit message: New model (world frame moved) New joint state node to capture joint states (se pick_callback)

File: ur_related/ur_manager_support/urdf/ur5_throw_cell.xacro (robot description, xacro)
@@ -180,6 +180,11 @@
     </joint>
     <!-- ***JOINTS*** -->
+    <!--<joint name="table_top_to_world" type="fixed"> OLD ONE
+        <origin xyz="0.625 0 0" rpy="0 0 0"/>
+        <parent link="world"/>
+        <child link="table_top"/>
+    </joint>-->
     <joint name="table_top_to_world" type="fixed">
-        <origin xyz="0.625 0 0" rpy="0 0 0"/>
+        <origin xyz="0.4955 0.4685 0" rpy="0 0 0"/>
         <parent link="world"/>
         <child link="table_top"/>
@@ -210,7 +215,12 @@
         <child link="camera"/>
     </joint>
-    <!-- robot link to world -->
+    <!-- robot link to world --> <!--OLD ONE-->
+    <!--<joint name="robot_to_world" type="fixed">
+        <origin xyz="0.1295 -0.4685 0" rpy="0 0 ${pi}"/>
+        <parent link="world"/>
+        <child link="base_link"/>
+    </joint>-->
     <joint name="robot_to_world" type="fixed">
-        <origin xyz="0.1295 -0.4685 0" rpy="0 0 ${pi}"/>
+        <origin xyz="0 0 0" rpy="0 0 ${pi}"/>
         <parent link="world"/>
         <child link="base_link"/>
